Commit message: urdf experiments

File: description/robot.urdf.xacro (robot description, xacro)
@@ -1,4 +1,11 @@
 <?xml version="1.0"?>
-<robot xmlns:xacro="http://www.ros.org/wiki/xacro"  name="robot">
-    <xacro:include filename="robot_core.xacro" />
+<robot name="vacuum_cleaner" xmlns:xacro="http://www.ros.org/wiki/xacro">
+    <xacro:property name="base_raduis"  value="0.175"/>
+    <xacro:property name="base_height"  value="0.100"/>
+    <xacro:property name="wheel_radius" value="0.035"/>
+    <xacro:property name="wheel_width"  value="0.025"/>
+    <xacro:property name="wheelbase"    value="0.250"/>
+    <xacro:property name="wheel_xoff"   value="-0.050"/>
+    <xacro:property name="wheel_zoff"   value="0.000"/>
+    <xacro:include filename="robot_core.xacro"/>
 </robot>

File: description/robot_core.xacro (robot description, xacro)
@@ -2,59 +2,33 @@
 <robot xmlns:xacro="http://www.ros.org/wiki/xacro">
 <link name="base_link">
-</link>
-<joint name="chassis_joint" type="fixed">
-    <parent link="base_link"/>
-    <child link="chassis"/>
-    <origin xyz="-0.1 0 0"/>
-</joint>
-<link name="chassis">
     <visual>
-        <origin xyz="0.15 0 0.075" rpy="0 0 0"/>
         <geometry>
-            <cylinder size="0.2 0.1"/>
+            <cylinder radius="${base_raduis}" length="${base_height}"/>
         </geometry>
-        <material name="white"/>
+        <material name="Cyan">
+            <color rgba="0 1.0 1.0 1.0"/>
+        </material>
     </visual>
 </link>
-<joint name="left_wheel_joint" type="continuous">
+<xacro:macro name="wheel" params="prefix y_reflect">
+  <link name="${prefix}_link">
+    <visual>
+      <origin xyz="0 0 0" rpy="${pi/2} 0 0"/>
+      <geometry>
+        <cylinder radius="${wheel_radius}" length="${wheel_width}"/>
+      </geometry>
+      <material name="Gray">
+        <color rgba="0.5 0.5 0.5 1.0"/>
+      </material>
+    </visual>
+  </link>
+  <joint name="${prefix}_joint" type="continuous">
     <parent link="base_link"/>
-    <child link="left_wheel"/>
-    <origin xyz="0 0.175 0" rpy="-${pi/2} 0 0"/>
-    <axis xyz="0 0 1"/>
-</joint>
-<link name="left_wheel">
-    <visual>
-        <geometry>
-            <cylinder length="0.04" radius="0.05" />
-        </geometry>
-        <material name="blue"/>
-    </visual>
-</link>
-<joint name="right_wheel_joint" type="continuous">
-    <parent link="base_link"/>
-    <child link="right_wheel"/>
-    <origin xyz="0 -0.175 0" rpy="${pi/2} 0 0"/>
-    <axis xyz="0 0 -1"/>
-</joint>
-<link name="right_wheel">
-    <visual>
-        <geometry>
-            <cylinder length="0.04" radius="0.05" />
-        </geometry>
-        <material name="blue"/>
-    </visual>
-</link>
-<joint name="caster_wheel_joint" type="fixed">
-    <parent link="chassis"/>
-    <child link="caster_wheel"/>
-    <origin xyz="0.24 0 0" rpy="0 0 0"/>
-</joint>
-<link name="caster_wheel">
-    <visual>
-        <geometry>
-            <sphere radius="0.05" />
-        </geometry>
-        <material name="black"/>
-    </visual>
-</link>
+    <child link="${prefix}_link"/>
+    <origin xyz="${wheel_xoff} ${y_reflect*(wheelbase/2)} ${-wheel_zoff}" rpy="0 0 0"/>
+    <axis xyz="0 1 0"/>
+  </joint>
+</xacro:macro>
+<xacro:wheel prefix="drive_wheel_l" y_reflect="1" />
+<xacro:wheel prefix="drive_wheel_r" y_reflect="-1" />
 </robot>

Commit message: urdf parametrization changes

File: description/robot.urdf.xacro (robot description, xacro)
@@ -7,5 +7,5 @@
     <xacro:property name="wheelbase"    value="0.250"/>
     <xacro:property name="wheel_xoff"   value="-0.050"/>
-    <xacro:property name="wheel_zoff"   value="0.000"/>
+    <xacro:property name="floor_gap"    value="0.020"/>
     <xacro:include filename="robot_core.xacro"/>
 </robot>

File: description/robot_core.xacro (robot description, xacro)
@@ -26,5 +26,5 @@
     <parent link="base_link"/>
     <child link="${prefix}_link"/>
-    <origin xyz="${wheel_xoff} ${y_reflect*(wheelbase/2)} ${-wheel_zoff}" rpy="0 0 0"/>
+    <origin xyz="${wheel_xoff} ${y_reflect*(wheelbase/2)} ${wheel_radius - base_height/2 + floor_gap}" rpy="0 0 0"/>
     <axis xyz="0 1 0"/>
   </joint>

Commit message: add caster wheel to urdf, some fixes

File: description/robot.urdf.xacro (robot description, xacro)
@@ -7,4 +7,5 @@
     <xacro:property name="wheelbase"    value="0.250"/>
     <xacro:property name="wheel_xoff"   value="-0.050"/>
+    <xacro:property name="caster_xoff"  value="0.100"/>
     <xacro:property name="floor_gap"    value="0.020"/>
     <xacro:include filename="robot_core.xacro"/>

File: description/robot_core.xacro (robot description, xacro)
@@ -11,4 +11,10 @@
     </visual>
 </link>
+<link name="base_footprint"/>
+<joint name="base_joint" type="fixed">
+  <parent link="base_link"/>
+  <child link="base_footprint"/>
+  <origin xyz="0.0 0.0 ${-base_height/2 - floor_gap}" rpy="0 0 0"/>
+</joint>
 <xacro:macro name="wheel" params="prefix y_reflect">
   <link name="${prefix}_link">
@@ -26,5 +32,5 @@
     <parent link="base_link"/>
     <child link="${prefix}_link"/>
-    <origin xyz="${wheel_xoff} ${y_reflect*(wheelbase/2)} ${wheel_radius - base_height/2 + floor_gap}" rpy="0 0 0"/>
+    <origin xyz="${wheel_xoff} ${y_reflect*(wheelbase/2)} ${wheel_radius - base_height/2 - floor_gap}" rpy="0 0 0"/>
     <axis xyz="0 1 0"/>
   </joint>
@@ -32,3 +38,18 @@
 <xacro:wheel prefix="drive_wheel_l" y_reflect="1" />
 <xacro:wheel prefix="drive_wheel_r" y_reflect="-1" />
+<link name="caster_link">
+  <visual>
+    <geometry>
+      <sphere radius="${floor_gap}"/>
+    </geometry>
+    <material name="Cyan">
+      <color rgba="0 1.0 1.0 1.0"/>
+    </material>
+  </visual>
+</link>
+<joint name="caster_joint" type="fixed">
+  <parent link="base_link"/>
+  <child link="caster_link"/>
+  <origin xyz="${caster_xoff} 0.0 ${-(base_height/2)}" rpy="0 0 0"/>
+</joint>
 </robot>
